File: DCMotorSpeedController.kicad_pcb (KiCad board)
At the start: 2 copper layers, 56.5 x 35.5 mm, 15 parts, among them J1 Motor Terminal, J2 Power Terminal, Q1 IRLZ44N, SW1 POWER_SW, U1 NE555P

Commit message: fixed diode position
Connections:
- C3 pad 1: Net-(D3-A) -> Net-(D3-K)
- J1 pad 1: Net-(D3-A) -> Net-(D3-K)
- J1 pad 2: Net-(D3-K) -> Net-(D3-A)
- Q1 pad 2: Net-(D3-K) -> Net-(D3-A)
- R1 pad 1: Net-(D3-A) -> Net-(D3-K)
- SW1 pad 2: Net-(D3-A) -> Net-(D3-K)
- U1 pad 4: Net-(D3-A) -> Net-(D3-K)
- U1 pad 8: Net-(D3-A) -> Net-(D3-K)
Changed lines of the file:
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@@
 			(crossoutdnponfab yes)
 			(subtractmaskfromsilk no)
-			(outputformat 1)
+			(outputformat 5)
 			(mirror no)
 			(drillshape 0)
@@
 			(remove_unused_layers no)
 			(roundrect_rratio 0.089286)
-			(net "Net-(D3-A)")
+			(net "Net-(D3-K)")
 			(pinfunction "Pin_1_1")
 			(pintype "passive")
@@
 			(layers "*.Cu" "*.Mask")
 			(remove_unused_layers no)
-			(net "Net-(D3-K)")
+			(net "Net-(D3-A)")
 			(pinfunction "Pin_2_2")
 			(pintype "passive")
@@
 			(layers "*.Cu" "*.Mask")
 			(remove_unused_layers no)
-			(net "Net-(D3-A)")
+			(net "Net-(D3-K)")
 			(pintype "passive")
 		)
@@
 			(remove_unused_layers no)
 			(roundrect_rratio 0.125)
-			(net "Net-(D3-A)")
+			(net "Net-(D3-K)")
 			(pintype "passive")
 		)
@@
 			(layers "*.Cu" "*.Mask")
 			(remove_unused_layers no)
-			(net "Net-(D3-K)")
+			(net "Net-(D3-A)")
 			(pinfunction "D_2")
 			(pintype "passive")
@@
 			(layers "*.Cu" "*.Mask")
 			(remove_unused_layers no)
-			(net "Net-(D3-A)")
+			(net "Net-(D3-K)")
 			(pinfunction "~{RST}_4")
 			(pintype "input")
@@
 			(layers "*.Cu" "*.Mask")
 			(remove_unused_layers no)
-			(net "Net-(D3-A)")
+			(net "Net-(D3-K)")
 			(pinfunction "VCC_8")
 			(pintype "power_in")
@@
 			(layers "*.Cu" "*.Mask")
 			(remove_unused_layers no)
-			(net "Net-(D3-A)")
+			(net "Net-(D3-K)")
 			(pinfunction "B_2")
 			(pintype "passive")
