File: DCMotorSpeedController.kicad_sch (KiCad schematic)
At the start: 15 parts, among them J1 Motor Terminal, J2 Power Terminal, Q1 IRLZ44N, SW1 POWER_SW, U1 NE555P

Commit message: more stuff
Parts:
- C1, C2, C3: KiLib_Generator (none) -> capacitor/THT/other
- D1, D2, D3: KiLib_Generator (none) -> diode/THT
- J1, J2: KiLib_Generator (none) -> terminal_block/MaiXu
- Q1: KiLib_Generator (none) -> package/TO_SOT/THT
- R1, R3, R4: KiLib_Generator (none) -> resistor/THT
- U1: KiLib_Generator (none) -> package/DIP/legacy
Other:
- moved on the sheet: C1, C2, C3, D1, D2, D3, J1, J2, Q1, R1, R3, R4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

Commit message: fixed diode position
Connections:
- net at J1.2 (Pin_2), Q1.2 (D): now also D3.2 (A); no longer D3.1 (K)
- net at C3.1, J1.1 (Pin_1), R1.1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: now also D3.1 (K); no longer D3.2 (A)
Other:
- moved on the sheet: D3
Changed lines of the file:
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@@
 	(symbol
 		(lib_id "Diode:1N4007")
-		(at 179.07 74.93 90)
+		(at 179.07 74.93 270)
 		(unit 1)
 		(body_style 1)
@@
 					(size 1.27 1.27)
 				)
-				(justify right)
+				(justify left)
 			)
 		)
@@
 					(size 1.27 1.27)
 				)
-				(justify right)
+				(justify left)
 			)
 		)
 		(property "Footprint" "Diode_THT:D_DO-41_SOD81_P10.16mm_Horizontal"
-			(at 183.515 74.93 0)
+			(at 174.625 74.93 0)
 			(hide yes)
 			(show_name no)
